File: i2c-keypad.kicad_pcb (KiCad board)
At the start: 2 copper layers, 21.4 x 34.7 mm, 10 parts, among them IC1 ATTINY84-S, P1 ICSP, P2 i2c, P3 PWR, P4 KEYPAD

Commit message: Added Image
Other:
- board text added: "https://github.com/mage0r/i2c-keypad Default address is 0x30 Copyright John Spencer, 2016"
- board text added: "i2c Keypad"
Changed lines of the file:
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@@
     (links 27)
     (no_connects 1)
-    (area 132.593999 92.048999 154.629001 127.588001)
+    (area 132.807639 92.546099 154.380001 127.405201)
     (thickness 1.6)
-    (drawings 22)
+    (drawings 24)
     (tracks 131)
     (zones 0)
@@
     (pad_to_mask_clearance 0.2)
     (aux_axis_origin 0 0)
-    (visible_elements FFFFFF7F)
+    (visible_elements 7FFFFFFF)
     (pcbplotparams
       (layerselection 0x010ff_80000001)
@@
     )
   )
+  (gr_text "i2c Keypad" (at 143.38808 108.1278) (layer B.SilkS)
+    (effects (font (size 1.5 1.5) (thickness 0.3)) (justify mirror))
+  )
+  (gr_text "https://github.com/mage0r/i2c-keypad\nDefault address is 0x30\nCopyright John Spencer, 2016" (at 144.11452 110.81004) (layer B.SilkS)
+    (effects (font (size 0.6 0.6) (thickness 0.15)) (justify mirror))
+  )
   (gr_text 9 (at 137.4648 119.5) (layer B.SilkS)

Commit message: Yep, ground plane.  caught again.
Routing:
- net /RST: track 39.0 -> 42.7 mm
- net +5V: track 35.0 -> 36.2 mm
Changed lines of the file:
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@@
-(kicad_pcb (version 4) (host pcbnew 4.0.2-stable)
+(kicad_pcb (version 4) (host pcbnew 4.0.4-stable)
   (general
     (links 27)
-    (no_connects 1)
-    (area 132.807639 92.546099 154.380001 127.405201)
+    (no_connects 0)
+    (area 132.593999 92.048999 154.652 127.588001)
     (thickness 1.6)
     (drawings 24)
@@
   (gr_line (start 132.88264 92.6211) (end 154.305 92.6211) (angle 90) (layer Edge.Cuts) (width 0.15))
   (gr_line (start 132.88264 127.3302) (end 132.88264 92.6211) (angle 90) (layer Edge.Cuts) (width 0.15))
+  (segment (start 134.569 103.022) (end 134.569 101.771) (width 0.25) (layer F.Cu) (net 1))
+  (segment (start 145.236 101.15) (end 147.02 102.934) (width 0.25) (layer F.Cu) (net 1))
+  (segment (start 135.19 101.15) (end 145.236 101.15) (width 0.25) (layer F.Cu) (net 1))
+  (segment (start 134.569 101.771) (end 135.19 101.15) (width 0.25) (layer F.Cu) (net 1))
   (segment (start 150.571 109.538) (end 150.571 107.861) (width 0.25) (layer F.Cu) (net 1))
   (segment (start 133.883 105.0493) (end 133.883 106.147) (width 0.25) (layer F.Cu) (net 1))
   (segment (start 134.569 104.3633) (end 133.883 105.0493) (width 0.25) (layer F.Cu) (net 1))
   (segment (start 134.569 103.022) (end 134.569 104.3633) (width 0.25) (layer F.Cu) (net 1))
-  (segment (start 135.9336 101.6574) (end 134.569 103.022) (width 0.25) (layer B.Cu) (net 1))
-  (segment (start 144.5545 101.6574) (end 135.9336 101.6574) (width 0.25) (layer B.Cu) (net 1))
-  (segment (start 145.8311 102.934) (end 144.5545 101.6574) (width 0.25) (layer B.Cu) (net 1))
-  (segment (start 147.02 102.934) (end 145.8311 102.934) (width 0.25) (layer B.Cu) (net 1))
   (segment (start 133.878 107.0488) (end 133.883 107.0438) (width 0.25) (layer F.Cu) (net 1))
   (segment (start 133.878 108.024) (end 133.878 107.0488) (width 0.25) (layer F.Cu) (net 1))
@@
   (segment (start 137.9017 106.106) (end 137.0343 106.106) (width 0.25) (layer F.Cu) (net 1))
   (segment (start 147.02 102.934) (end 148.1064 102.934) (width 0.25) (layer F.Cu) (net 1))
+  (segment (start 150.571 107.861) (end 150.571 107.1547) (width 0.25) (layer F.Cu) (net 1))
+  (segment (start 148.1064 102.934) (end 148.1064 103.1705) (width 0.25) (layer F.Cu) (net 1))
+  (segment (start 148.1064 103.1705) (end 149.2068 104.2709) (width 0.25) (layer F.Cu) (net 1))
+  (segment (start 149.2068 104.2709) (end 150.0397 104.2709) (width 0.25) (layer F.Cu) (net 1))
+  (segment (start 150.0397 104.2709) (end 150.7651 104.9963) (width 0.25) (layer F.Cu) (net 1))
+  (segment (start 150.7651 104.9963) (end 150.7651 106.9606) (width 0.25) (layer F.Cu) (net 1))
   (segment (start 150.7651 106.9606) (end 150.571 107.1547) (width 0.25) (layer F.Cu) (net 1))
-  (segment (start 150.7651 104.9963) (end 150.7651 106.9606) (width 0.25) (layer F.Cu) (net 1))
-  (segment (start 150.0397 104.2709) (end 150.7651 104.9963) (width 0.25) (layer F.Cu) (net 1))
-  (segment (start 149.2068 104.2709) (end 150.0397 104.2709) (width 0.25) (layer F.Cu) (net 1))
-  (segment (start 148.1064 103.1705) (end 149.2068 104.2709) (width 0.25) (layer F.Cu) (net 1))
-  (segment (start 148.1064 102.934) (end 148.1064 103.1705) (width 0.25) (layer F.Cu) (net 1))
-  (segment (start 150.571 107.861) (end 150.571 107.1547) (width 0.25) (layer F.Cu) (net 1))
   (via (at 152.3646 113.8918) (size 0.6) (layers F.Cu B.Cu) (net 2))
   (via (at 144.6155 105.964) (size 0.6) (layers F.Cu B.Cu) (net 2))
@@
   (segment (start 133.2276 108.7633) (end 134.3803 109.916) (width 0.25) (layer F.Cu) (net 6))
   (segment (start 133.2276 101.8481) (end 133.2276 108.7633) (width 0.25) (layer F.Cu) (net 6))
-  (segment (start 133.876 101.1997) (end 133.2276 101.8481) (width 0.25) (layer F.Cu) (net 6))
-  (segment (start 152.0471 101.1997) (end 133.876 101.1997) (width 0.25) (layer F.Cu) (net 6))
-  (segment (start 153.2889 102.4415) (end 152.0471 101.1997) (width 0.25) (layer F.Cu) (net 6))
+  (segment (start 133.756 99.1097) (end 133.2276 101.8481) (width 0.25) (layer F.Cu) (net 6))
+  (segment (start 151.9271 99.1097) (end 133.756 99.1097) (width 0.25) (layer F.Cu) (net 6))
+  (segment (start 153.2889 102.4415) (end 151.9271 99.1097) (width 0.25) (layer F.Cu) (net 6))
   (segment (start 153.2889 103.4265) (end 153.2889 102.4415) (width 0.25) (layer F.Cu) (net 6))
   (segment (start 152.4303 104.2851) (end 153.2889 103.4265) (width 0.25) (layer F.Cu) (net 6))
